File: Power.kicad_sch (KiCad schematic)
At the start: 3 parts, among them J5 VCC_IN

Commit message: rev v3 tiny
Parts:
- J5: footprint Connector_AMASS:AMASS_XT60PW-M_1x02_P7.20mm_Horizontal -> lib:XT60-RightAngle-Adapter
Connections:
- net GND: now also J5.2 (Pin_2); no longer J5.1 (Pin_1)
- net VCC: now also J5.1 (Pin_1); no longer J5.2 (Pin_2)
Changed lines of the file:
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@@
 	(symbol
 		(lib_id "Connector_Generic:Conn_01x02")
-		(at 128.27 80.01 0)
-		(mirror x)
+		(at 128.27 77.47 0)
 		(unit 1)
 		(exclude_from_sim no)
@@
 		(dnp no)
 		(property "Reference" "J5"
-			(at 130.81 80.0101 0)
+			(at 130.81 77.4699 0)
 			(effects
 				(font
@@
 		)
 		(property "Value" "VCC_IN"
-			(at 130.81 77.4701 0)
+			(at 130.81 80.0099 0)
 			(effects
 				(font
@@
 			)
 		)
-		(property "Footprint" "Connector_AMASS:AMASS_XT60PW-M_1x02_P7.20mm_Horizontal"
-			(at 128.27 80.01 0)
+		(property "Footprint" "lib:XT60-RightAngle-Adapter"
+			(at 128.27 77.47 0)
 			(effects
 				(font
@@
 		)
 		(property "Datasheet" "~"
-			(at 128.27 80.01 0)
+			(at 128.27 77.47 0)
 			(effects
 				(font
@@
 		)
 		(property "Description" "Generic connector, single row, 01x02, script generated (kicad-library-utils/schlib/autogen/connector/)"
-			(at 128.27 80.01 0)
+			(at 128.27 77.47 0)
 			(effects
 				(font
@@
 		)
 		(instances
-			(project "vesc_mms_board"
+			(project "ModuCard-vesc-to-mms-converter"
 				(path "/19c3ad7a-1b7d-4298-9053-cf734bfcea10/09185991-2b08-4e41-9e65-0618febadbdd"
 					(reference "J5")
