File: can.kicad_sch (KiCad schematic)
At the start: 14 parts, among them J1 RJ45_LED_Shielded, J2 RJ45_LED_Shielded, J3 Conn_01x04, SW1 SW_DIP_x02

Commit message: rev v3 tiny
Parts:
- removed J1, J2: RJ45_LED_Shielded, Connector_RJ:RJ45_Amphenol_RJHSE538X, symbol Connector:RJ45_LED_Shielded
- removed R1, R17, R18, R4: 1k, Resistor_SMD:R_0402_1005Metric, symbol Device:R
- removed R2, R3: 120R, Resistor_SMD:R_0603_1608Metric, symbol Device:R
- removed R5, R6, R7, R8: 0R, Resistor_SMD:R_0603_1608Metric, symbol Device:R
- added R1, R4, R5, R6: 0Ω, PCM_JLCPCB:R_0402, symbol PCM_JLCPCB-Resistors:0402,0Ω
- added R15, R16, R19, R20: 1k, Resistor_SMD:R_0402_1005Metric, symbol Device:R
- added R2, R7: 120Ω, PCM_JLCPCB:R_0402, symbol PCM_JLCPCB-Resistors:0402,120Ω
- added U2: XDRJ-1609-002, rj45:RJ45-TH_XDRJ-1609-002, symbol rj45:XDRJ-1609-002
Connections:
- net +12V: now also R15.2, R16.2, R19.2, R20.2, U2.14, U2.6
- net CAN+: now also R1.2, R5.1
- net CAN-: now also R4.2, R6.1
- net CAN1+: now also R1.1, R2.1, U2.10, U2.2; no longer SW1.4
- net CAN1-: now also SW1.3, R4.1, U2.1, U2.9
- net CAN2+: now also R5.2, R7.1, U2.13, U2.5
- net CAN2-: now also SW1.4, R6.2, U2.12, U2.4; no longer SW1.3
- net GND: now also U2.11, U2.17 (-), U2.19 (-), U2.21 (-), U2.23 (-), U2.25, U2.26, U2.27, U2.28, U2.29, U2.3, U2.30
- net USB_DOWNSTREAM_D+: now also U2.16
- net USB_DOWNSTREAM_D-: now also U2.15
- net USB_UPSTREAM_D+: now also U2.8
- net USB_UPSTREAM_D-: now also U2.7
- net at SW1.2: now also R2.2
- net at SW1.1: now also R7.2
- new net: R16.1, U2.20 (+)
- new net: R19.1, U2.22 (+)
- new net: R15.1, U2.18 (+)
- new net: R20.1, U2.24 (+)
Other:
- note removed: "PASS THROUYH BUS CONENCTOR"
- moved on the sheet: J3

Commit message: rev 1
Connections:
- net +12V: now also U2.22 (+); no longer R19.2
- net GND: now also R19.2; no longer U2.21 (-)
- net at R19.1: now also U2.21 (-); no longer U2.22 (+)
Other:
- moved on the sheet: R19
Changed lines of the file:
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@@
+	(wire
+		(pts
+			(xy 146.05 107.95) (xy 148.59 107.95)
+		)
+		(stroke
+			(width 0)
+			(type default)
+		)
+	)
 	(wire
 		(pts
@@
 	(wire
 		(pts
-			(xy 146.05 107.95) (xy 148.59 107.95)
-		)
-		(stroke
-			(width 0)
-			(type default)
-		)
-	)
-	(wire
-		(pts
 			(xy 163.83 36.83) (xy 163.83 44.45)
 		)
@@
 	(wire
 		(pts
-			(xy 157.48 109.22) (xy 157.48 110.49)
+			(xy 163.83 109.22) (xy 163.83 110.49)
 		)
 		(stroke
@@
 	(wire
 		(pts
+			(xy 156.21 107.95) (xy 158.75 107.95)
+		)
+		(stroke
+			(width 0)
+			(type default)
+		)
+	)
+	(wire
+		(pts
 			(xy 158.75 55.88) (xy 158.75 60.96)
 		)
@@
 	(wire
 		(pts
-			(xy 146.05 110.49) (xy 149.86 110.49)
+			(xy 146.05 110.49) (xy 163.83 110.49)
 		)
 		(stroke
@@
 	(symbol
 		(lib_id "Device:R")
-		(at 153.67 110.49 90)
+		(at 152.4 107.95 90)
 		(unit 1)
 		(exclude_from_sim no)
@@
 		(dnp no)
 		(property "Reference" "R19"
-			(at 152.4 111.76 0)
+			(at 151.13 109.22 0)
 			(effects
 				(font
@@
 		)
 		(property "Value" "1k"
-			(at 154.94 111.76 0)
+			(at 153.67 109.22 0)
 			(effects
 				(font
@@
 		)
 		(property "Footprint" "Resistor_SMD:R_0402_1005Metric"
-			(at 153.67 112.268 90)
+			(at 152.4 109.728 90)
 			(effects
 				(font
@@
 		)
 		(property "Datasheet" "~"
-			(at 153.67 110.49 0)
+			(at 152.4 107.95 0)
 			(effects
 				(font
@@
 		)
 		(property "Description" ""
-			(at 153.67 110.49 0)
+			(at 152.4 107.95 0)
 			(effects
 				(font
@@
 	(symbol
 		(lib_id "power:+12V")
-		(at 157.48 109.22 0)
+		(at 163.83 109.22 0)
 		(unit 1)
 		(exclude_from_sim no)
@@
 		(fields_autoplaced yes)
 		(property "Reference" "#PWR032"
-			(at 157.48 113.03 0)
+			(at 163.83 113.03 0)
 			(effects
 				(font
@@
 		)
 		(property "Value" "+12V"
-			(at 157.48 104.14 0)
+			(at 163.83 104.14 0)
 			(effects
 				(font
@@
 		)
 		(property "Footprint" ""
-			(at 157.48 109.22 0)
+			(at 163.83 109.22 0)
 			(effects
 				(font
@@
 		)
 		(property "Datasheet" ""
-			(at 157.48 109.22 0)
+			(at 163.83 109.22 0)
 			(effects
 				(font
@@
 		)
 		(property "Description" "Power symbol creates a global label with name \"+12V\""
-			(at 157.48 109.22 0)
+			(at 163.83 109.22 0)
 			(effects
 				(font
@@
 	(symbol
 		(lib_id "power:GND")
-		(at 148.59 107.95 90)
+		(at 158.75 107.95 90)
 		(unit 1)
 		(exclude_from_sim no)
@@
 		(dnp no)
 		(property "Reference" "#PWR036"
-			(at 154.94 107.95 0)
+			(at 165.1 107.95 0)
 			(effects
 				(font
@@
 		)
 		(property "Value" "GND"
-			(at 152.4 107.95 0)
+			(at 162.56 107.95 0)
 			(effects
 				(font
@@
 		)
 		(property "Footprint" ""
-			(at 148.59 107.95 0)
+			(at 158.75 107.95 0)
 			(effects
 				(font
@@
 		)
 		(property "Datasheet" ""
-			(at 148.59 107.95 0)
+			(at 158.75 107.95 0)
 			(effects
 				(font
@@
 		)
 		(property "Description" ""
-			(at 148.59 107.95 0)
-			(effects
-				(font
+			(at 158.75 107.95 0)
+			(effects
+				(font

Commit message: fix chinczyk funckup
Parts:
- removed R1, R4, R5, R6: 0Ω, PCM_JLCPCB:R_0402, symbol PCM_JLCPCB-Resistors:0402,0Ω
- removed R2, R7: 120Ω, PCM_JLCPCB:R_0402, symbol PCM_JLCPCB-Resistors:0402,120Ω
- added R1, R3, R4, R5: 0Ω, PCM_JLCPCB:R_0603, symbol PCM_JLCPCB-Resistors:0603,0Ω
- added R2, R6: 120Ω, PCM_JLCPCB:R_0603, symbol PCM_JLCPCB-Resistors:0603,120Ω
Connections:
- net +12V: now also U2.3; no longer U2.6
- net CAN+: now also R1.2, R4.1
- net CAN-: now also R3.2, R5.1
- net CAN1+: now also SW1.4, U2.7, R1.1; no longer U2.2
- net CAN1-: now also U2.8, R3.1, R6.1; no longer SW1.3, U2.1
- net CAN2+: now also U2.4, R2.2, R4.2; no longer U2.5
- net CAN2-: now also SW1.3, U2.5, R5.2; no longer SW1.4, U2.4
- net GND: now also U2.6; no longer U2.3
- net USB_UPSTREAM_D+: now also U2.1; no longer U2.8
- net USB_UPSTREAM_D-: now also U2.2; no longer U2.7
- net at SW1.2: now also R2.1
- net at SW1.1: now also R6.2
